Commit message: Add files via upload

File: rw/model/robot.xacro (robot description, xacro)
@@ -1,23 +1,21 @@
 <?xml version="1.0"?>
-<robot name="rw" xmlns:xacro="http://www.ros.org/wiki/xacro">
+<robot name="rw_bot" xmlns:xacro="http://www.ros.org/wiki/xacro">
     <xacro:property name="PI" value="3.14159265"/>
-    <material name="white">
-        <color rgba="1 1 1 1" />
-    </material>
-    <material name="gray">
-        <color rgba="0.7529 0.7529 0.7529 1"/>
-    </material>
-    <material name="blue">
-        <color rgba="0.2 0.2 1 1"/>E
-    </material>
-    <material name="black">
-        <color rgba="0 0 0 1"/>
-    </material>
-    <material name="red">
-        <color rgba="1 0 0 1"/>
-    </material>
-    <!-- Control Parameters -->
-    <xacro:property name="max_linear_acceleration" value="20"/>
+    <xacro:property name="wheel_radius" value="0.113"/>
+    <xacro:property name="wheel_separation" value="0.554"/>
+    <!-- MATERIALS -->
+    <material name="white"> <color rgba="1 1 1 1"/> </material>
+    <material name="gray"> <color rgba="0.7529 0.7529 0.7529 1"/> </material>
+    <material name="blue"> <color rgba="0.2 0.2 1 1"/> </material>
+    <material name="black"> <color rgba="0 0 0 1"/> </material>
+    <material name="red"> <color rgba="1 0 0 1"/> </material>
+    <!-- Robot footprint -->
+    <link name="base_footprint"></link>
     <!-- Body Link -->
+    <joint name="base_footprint_joint" type="fixed">
+        <origin xyz="0 0 0" rpy="0 0 0" />
+        <parent link="base_footprint"/>
+        <child link="base_link" />
+    </joint>
     <link name="base_link">
         <visual>
@@ -33,23 +31,12 @@
                 <mesh filename="file://$(find rw)/meshes/base_link.stl" />
             </geometry>
-            <material name="gray"/>
-        </collision>
-        <inertial>
-            <mass value="1000"/>
-            <inertia ixx="0.5" ixy="0.0" ixz="0.0" iyy="0.5" iyz="0.0" izz="0.5"/>
-            <origin xyz="0 0 0" rpy="0 0 0"/>
-        </inertial>
-    </link>
-    <gazebo reference="base_link">
-        <mu1>1.0</mu1>
-        <mu2>1.0</mu2>
-    </gazebo>
-    <!-- BASE_FOOTPRINT LINK -->
-    <joint name="base_footprint_joint" type="fixed">
-        <origin xyz="0 0 0" rpy="0 0 0"/>
-        <parent link="base_link"/>
-        <child link="base_footprint"/>
-    </joint>
-    <link name="base_footprint">
+        </collision>
+        <inertial>
+            <mass value="62.4811"/>
+            <origin xyz="0.236253 0.0 0.191338" rpy="0 0 0"/>
+            <inertia ixx="5.98616" ixy="-0.000042" ixz="-2.594206"
+                     iyy="7.61358" iyz="0.000042"
+                     izz="6.642833"/>
+        </inertial>
     </link>
     <!-- Left Wheel -->
@@ -67,24 +54,22 @@
                 <mesh filename="file://$(find rw)/meshes/left_wheel.stl" />
             </geometry>
-            <material name="black"/>
-        </collision>
-        <inertial>
-            <mass value="200"/>
-            <inertia ixx="0.1" ixy="0.0" ixz="0.0" iyy="0.1" iyz="0.0" izz="0.2"/>
-            <origin xyz="0.0 0.0 0.0" rpy="0.0 0.0 0.0"/>
+        </collision>
+        <inertial>
+            <mass value="0.4545"/>
+            <origin xyz="0.000001  0.024997 -0.000001" rpy="0.0 0.0 0.0"/>
+            <inertia ixx="0.002609" ixy="0.0" ixz="0.0"
+                     iyy="0.005028" iyz="0.0"
+                     izz="0.002609"/>
         </inertial>
     </link>
     <joint name="wheel_left_joint" type="continuous">
-        <origin xyz="0 -0.2772 0" rpy="0 0 0" />
+        <origin xyz="0.0 ${wheel_separation/2} 0" rpy="0 0 0" />
         <parent link="base_link"/>
         <child link="wheel_left_link"/>
         <axis xyz="0 1 0"/>
-        <limit effort="100" velocity="300.0"/>
-        <dynamics damping="1" friction="10"/>
-    </joint>
-    <gazebo reference="wheel_left_link">
-        <mu1>1.0</mu1>
-        <mu2>1.0</mu2>
-    </gazebo>
+        <limit effort="50" velocity="62"/>
+        <dynamics damping="0.1" friction="0.1"/>
+    </joint>
+    <gazebo reference="wheel_left_link"> <mu1>1.0</mu1> <mu2>1.0</mu2> <material>Gazebo/Black</material> </gazebo>
     <!-- right Wheel -->
     <link name="wheel_right_link">
@@ -101,24 +86,22 @@
                 <mesh filename="file://$(find rw)/meshes/right_wheel.stl" />
             </geometry>
-            <material name="black"/>
-        </collision>
-        <inertial>
-            <mass value="200"/>
-            <inertia ixx="0.1" ixy="0.0" ixz="0.0" iyy="0.1" iyz="0.0" izz="0.2"/>
-            <origin xyz="0.0 0.0 0.0" rpy="0.0 0.0 0.0"/>
+        </collision>
+        <inertial>
+            <mass value="0.4545"/>
+            <origin xyz="0.000001  0.024997 -0.000001" rpy="0.0 0.0 0.0"/>
+            <inertia ixx="0.002609" ixy="0.0" ixz="0.0"
+                     iyy="0.005028" iyz="0.0"
+                     izz="0.002609"/>
         </inertial>
     </link>
     <joint name="wheel_right_joint" type="continuous">
-        <origin xyz="0.0 0.2772 0" rpy="0 0 0" />
+        <origin xyz="0.0 ${-wheel_separation/2} 0" rpy="0 0 0" />
         <parent link="base_link"/>
         <child link="wheel_right_link"/>
         <axis xyz="0 1 0"/>
-        <limit effort="100" velocity="300.0"/>
-        <dynamics damping="1" friction="10"/>
-    </joint>
-    <gazebo reference="wheel_right_link">
-        <mu1>1.0</mu1>
-        <mu2>1.0</mu2>
-    </gazebo>
+        <limit effort="50" velocity="62"/>
+        <dynamics damping="0.1" friction="0.1"/>
+    </joint>
+    <gazebo reference="wheel_right_link"> <mu1>1.0</mu1> <mu2>1.0</mu2> <material>Gazebo/Black</material> </gazebo>
     <!-- FRONT LEFT CASTER WHEEL LINK -->
     <link name="front_left_caster_wheel_link">
@@ -135,20 +118,23 @@
                 <sphere radius="0.11"/>
             </geometry>
-            <material name="black"/>
-        </collision>
-        <inertial>
-            <mass value="50"/>
-            <inertia ixx="0.0002" ixy="0.0" ixz="0.0" iyy="0.01" iyz="0.0" izz="0.0002"/>
-            <origin xyz="0 0 0" rpy="0 0 0"/>
+        </collision>
+        <inertial>
+            <mass value="0.2461"/>
+            <origin xyz="0.018399  0.000732 -0.044236" rpy="0.0 0.0 0.0"/>
+            <!-- Inertia estimated via scaling Aluminum results -->
+            <inertia ixx="0.000285" ixy="-0.000001" ixz="0.000034"
+                     iyy="0.000382" iyz="0.000004"
+                     izz="0.000169"/>
         </inertial>
     </link>
     <joint name="front_left_caster_wheel_joint" type="fixed">
-        <origin xyz="-0.6490525 -0.2152957 -0.0024993" rpy="0 0 0"/>
+        <origin xyz="0.6490525 0.2152957 -0.0024993" rpy="0 0 0"/>
         <parent link="base_link"/>
         <child link="front_left_caster_wheel_link"/>
+        <dynamics damping="0.1" friction="0.1"/>
     </joint>
     <gazebo reference="front_left_caster_wheel_link">
-        <mu1>0.01</mu1>
-        <mu2>0.01</mu2>
+        <mu1>0.1</mu1>
+        <mu2>0.1</mu2>
     </gazebo>
     <!-- FRONT RIGHT CASTER WHEEL -->
@@ -169,17 +155,21 @@
         </collision>
         <inertial>
-            <mass value="50"/>
-            <inertia ixx="0.0002" ixy="0.0" ixz="0.0" iyy="0.01" iyz="0.0" izz="0.0002"/>
-            <origin xyz="0 0 0" rpy="0 0 0"/>
+            <mass value="0.2461"/>
+            <origin xyz="0.018399  0.000732 -0.044236" rpy="0.0 0.0 0.0"/>
+            <!-- Inertia estimated via scaling Aluminum results -->
+            <inertia ixx="0.000285" ixy="-0.000001" ixz="0.000034"
+                     iyy="0.000382" iyz="0.000004"
+                     izz="0.000169"/>
         </inertial>
     </link>
     <joint name="front_right_caster_wheel_joint" type="fixed">
-        <origin xyz="-0.6490525 0.2152957 -0.0024993" rpy="0 0 0"/>
+        <origin xyz="0.6490525 -0.2152957 -0.0024993" rpy="0 0 0"/>
         <parent link="base_link"/>
         <child link="front_right_caster_wheel_link"/>
+        <dynamics damping="0.1" friction="0.1"/>
     </joint>
     <gazebo reference="front_right_caster_wheel_link">
-        <mu1>0.01</mu1>
-        <mu2>0.01</mu2>
+        <mu1>0.1</mu1>
+        <mu2>0.1</mu2>
     </gazebo>
     <!-- Back CAMERA -->
@@ -202,14 +192,20 @@
         <parent link="base_link"/>
         <child link="back_camera_link"/>
-        <origin xyz="0.0431295 0 0.1042074" rpy="0 0 0"/>
-    </joint>
-    <link name="back_camera_link_optical"></link>
+        <origin xyz="-0.0431295 0 0.1042074" rpy="0 0 0"/>
+    </joint>
+    <link name="back_camera_link_optical">
+        <inertial>
+            <mass value="0.001" />
+            <origin xyz="0 0 0" rpy="0 0 0" />
+            <inertia ixx="1e-9" ixy="0" ixz="0" iyy="1e-9" iyz="0" izz="1e-9" />
+        </inertial>
+    </link>
     <joint name="back_camera_optical_joint" type="fixed">
         <parent link="back_camera_link"/>
         <child link="back_camera_link_optical"/>
-        <origin xyz="0.0621685 0 -0.0048553" rpy="0 ${pi/4} 0"/>
+        <origin xyz="-0.0621685 0 -0.0048553" rpy="0 ${3*pi/4} 0"/>
     </joint>
     <gazebo reference="back_camera_link_optical">
-        <sensor name="rgbd_camera" type="rgbd_camera">
+        <sensor name="back_rgbd_camera" type="rgbd_camera">
         <camera>
             <horizontal_fov>1.9</horizontal_fov>
@@ -222,4 +218,6 @@
             <far>1</far>
             </clip>
+            <!-- No need for this line anymore, Gazebo will use the reference frame -->
+            <!-- <optical_frame_id>back_camera_link_optical</optical_frame_id> -->
             <optical_frame_id>back_camera_link_optical</optical_frame_id>
         </camera>
@@ -228,5 +226,7 @@
         <visualize>true</visualize>
         <topic>camera2</topic>
-        <gz_frame_id>back_camera_link</gz_frame_id>
+        <!-- CHANGE THIS LINE -->
+        <!-- FROM: <gz_frame_id>back_camera_link</gz_frame_id> -->
+        <!--   TO: This will now implicitly use the "reference" link, which is correct -->
         </sensor>
     </gazebo>
@@ -248,21 +248,19 @@
         </collision>
         <inertial>
-            <mass value="2"/>
-            <inertia ixx="0.1" ixy="0.0" ixz="0.0" iyy="0.1" iyz="0.0" izz="0.2"/>
-            <origin xyz="0.0 0.0 0.0" rpy="0.0 0.0 0.0"/>
+            <mass value="0.2461"/>
+            <origin xyz="0.0 -0.0 0.005" rpy="0.0 0.0 0.0"/>
+            <inertia ixx="0.000003" ixy="-0.0" ixz="0.0"
+                     iyy="0.000003" iyz="0.0"
+                     izz="0.000006"/>
         </inertial>
     </link>
     <joint name="panAndTile_kit_joint" type="continuous">
-        <origin xyz="-0.6622757 0.0 0.7159456" rpy="0 0 0" />
+        <origin xyz="0.6622757 0.0 0.7159456" rpy="0 ${pi/8} 0" />
         <parent link="base_link"/>
         <child link="panAndTile_kit"/>
         <axis xyz="0 0 1"/>
-        <limit effort="100" velocity="300.0"/>
+        <limit effort="1" velocity="3.0"/>
         <dynamics damping="1" friction="1"/>
     </joint>
-    <gazebo reference="panAndTile_kit">
-        <mu1>1.0</mu1>
-        <mu2>1.0</mu2>
-    </gazebo>
     <!-- front CAMERA -->
     <link name="front_camera_link">
@@ -290,32 +288,32 @@
         <parent link="front_camera_link"/>
         <child link="front_camera_link_optical"/>
-        <origin xyz="-0.0202968 0 0.0228071" rpy="0 -${pi} 0"/>
+        <origin xyz="0.0202968 0 0.0228071" rpy="0.0 0.0 0.0"/>
     </joint>
     <gazebo reference="front_camera_link_optical">
-        <sensor name="rgbd_camera" type="rgbd_camera">
-        <camera>
-            <horizontal_fov>1.25</horizontal_fov>
-            <image>
-            <width>640</width>
-            <height>480</height>
-            </image>
-            <clip>
-            <near>0.3</near>
-            <far>15</far>
-            </clip>
-            <optical_frame_id>front_camera_link_optical</optical_frame_id>
-        </camera>
-        <always_on>1</always_on>
-        <update_rate>20</update_rate>
-        <visualize>true</visualize>
-        <topic>camera</topic>
-        <gz_frame_id>front_camera_link</gz_frame_id>
+        <sensor name="front_rgbd_camera" type="rgbd_camera">
+            <camera>
+                <horizontal_fov>1.25</horizontal_fov>
+                <image>
+                    <width>640</width>
+                    <height>480</height>
+                </image>
+                <clip>
+                    <near>0.3</near>
+                    <far>15</far>
+                </clip>
+                <!-- THIS IS THE CORRECT TAG AND LOCATION -->
+                <optical_frame_id>front_camera_link_optical</optical_frame_id>
+            </camera>
+            <always_on>1</always_on>
+            <update_rate>20</update_rate>
+            <visualize>true</visualize>
+            <topic>camera</topic>
         </sensor>
     </gazebo>
-    <!-- LIDAR -->
-    <link name="laser_frame">
-        <visual>
-            <geometry>
-                <mesh filename="file://$(find rw)/meshes/lidar.stl" />
+    <!-- Front LIDAR -->
+    <link name="front_laser_frame">
+        <visual>
+            <geometry>
+                <mesh filename="file://$(find rw)/meshes/front_lidar.stl" />
             </geometry>
             <material name="white"/>
@@ -323,5 +321,5 @@
         <collision>
             <geometry>
-                <mesh filename="file://$(find rw)/meshes/lidar.stl" />
+                <mesh filename="file://$(find rw)/meshes/front_lidar.stl" />
             </geometry>
             <material name="white"/>
@@ -330,36 +328,99 @@
     <joint name="laser_joint" type="fixed">
         <parent link="panAndTile_kit"/>
-        <child link="laser_frame"/>
+        <child link="front_laser_frame"/>
         <origin xyz="0.0 0.0 0.0556141" rpy="0 0 0"/>
     </joint>
-    <link name="lidar_link_optical"></link>
+    <link name="front_lidar_link_optical"></link>
     <joint name="lidar_optical_joint" type="fixed">
-        <parent link="laser_frame"/>
-        <child link="lidar_link_optical"/>
-        <origin xyz="-0.025 0 0.03" rpy="0 -${pi} 0"/>
-    </joint>
-    <gazebo reference="lidar_link_optical">
+        <parent link="front_laser_frame"/>
+        <child link="front_lidar_link_optical"/>
+        <origin xyz="0.025 0 0.03" rpy="0.0 0.0 0.0"/>
+    </joint>
+    <gazebo reference="front_lidar_link_optical">
         <sensor name="gpu_lidar" type="gpu_lidar">
-            <update_rate>30</update_rate>
-            <topic>scan</topic>
-            <gz_frame_id>lidar_link_optical</gz_frame_id>
+            <update_rate>10</update_rate>
+            <topic>scan_02</topic>
+            <gz_frame_id>front_lidar_link_optical</gz_frame_id>
             <lidar>
                 <scan>
                 <horizontal>
-                    <samples>50</samples>
+                    <samples>175</samples>
                     <!--(max_angle-min_angle)/samples * resolution -->
                     <resolution>1</resolution>
-                    <min_angle>${-pi/4}</min_angle>
-                    <max_angle>${pi/4}</max_angle>
+                    <min_angle>-0.61086523819</min_angle>
+                    <max_angle>0.61086523819</max_angle>
                 </horizontal>
                 <!-- Dirty hack for fake lidar detections with ogre 1 rendering in VM -->
                 <vertical>
                     <samples>50</samples>
-                    <min_angle>${-pi/4}</min_angle>
-                    <max_angle>${pi/8}</max_angle>
+                    <min_angle>-0.26179938779</min_angle>
+                    <max_angle>0.26179938779</max_angle>
                 </vertical>
                 </scan>
                 <range>
-                <min>0.05</min>
+                <min>1.5</min>
+                <max>75</max>
+                <resolution>0.01</resolution>
+                </range>
+                <noise>
+                    <type>gaussian</type>
+                    <mean>0.0</mean>
+                    <stddev>0.01</stddev>
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